Commit message: NED to ENU transform

File: src/state_estimation/urdf/robot.xacro (robot description, xacro)
@@ -83,5 +83,5 @@
     </gazebo>
     <!-- a link aligned with the steer direction -->
-    <joint name="steer_joint" type="revolute" >
+    <joint name="steer_joint" type="fixed" >
         <limit lower="-0.5" upper="0.5" effort="100" velocity="10" />
         <axis xyz="0 0 1" />
@@ -114,5 +114,5 @@
     </gazebo>
     <!-- the left Ackermann bar -->
-    <joint name="front_left_bar_joint" type="revolute" >
+    <joint name="front_left_bar_joint" type="fixed" >
         <limit lower="-0.5" upper="0.5" effort="100" velocity="10" />
         <axis xyz="0 0 1" />
@@ -145,5 +145,5 @@
     </gazebo>
     <!-- the right Ackermann bar -->
-    <joint name="front_right_bar_joint" type="revolute" >
+    <joint name="front_right_bar_joint" type="fixed" >
         <limit lower="-0.5" upper="0.5" effort="100" velocity="10" />
         <axis xyz="0 0 1" />
@@ -176,5 +176,5 @@
     </gazebo>
 	<!-- the front left wheel -->
-    <joint name="front_left_wheel_joint" type="continuous" >
+    <joint name="front_left_wheel_joint" type="fixed" >
         <axis xyz="0 1 0" />
         <parent link="front_left_bar_link" />
@@ -206,5 +206,5 @@
     </gazebo>
 	<!-- the front right wheel -->
-    <joint name="front_right_wheel_joint" type="continuous" >
+    <joint name="front_right_wheel_joint" type="fixed" >
         <axis xyz="0 1 0" />
         <parent link="front_right_bar_link" />
@@ -237,5 +237,5 @@
     </gazebo>
 	<!-- the Ackerman bar -->
-    <joint name="ackermann_joint" type="revolute" >
+    <joint name="ackermann_joint" type="fixed" >
         <limit lower="-0.5" upper="0.5" effort="100" velocity="10" />
         <axis xyz="0 0 1" />
@@ -288,5 +288,5 @@
     </gazebo>
 	<!-- the back left wheel -->
-    <joint name="back_left_wheel_joint" type="continuous" >
+    <joint name="back_left_wheel_joint" type="fixed" >
         <axis xyz="0 1 0" />
         <parent link="base_link" />
@@ -318,5 +318,5 @@
     </gazebo>
 	<!-- the back right wheel -->
-    <joint name="back_right_wheel_joint" type="continuous" >
+    <joint name="back_right_wheel_joint" type="fixed" >
         <axis xyz="0 1 0" />
         <parent link="base_link" />
@@ -404,5 +404,5 @@
         </link>
         <joint name="radar_joint" type="fixed" >
-            <origin xyz="0.0275 0 0.005" rpy="0 ${M_PI/2} 0" />
+            <origin xyz="0.0275 0 0.005" rpy="${M_PI/2} 0 0" />
             <parent link="sensors_base_link" />
             <child link="radar_link"/>
@@ -416,5 +416,5 @@
             <origin xyz="0 0 0.0275" rpy="0 0 0" />
             <parent link="sensors_base_link" />
-            <child link="gnss_link"/>
+            <child link="gps_link"/>
         </joint>
         <link name="radar_link">
@@ -456,5 +456,5 @@
             </collision>
         </link>
-        <link name="gnss_link">
+        <link name="gps_link">
             <inertial>
                 <mass value="0.1"/>
@@ -484,5 +484,5 @@
             <material>Gazebo/Red</material>
         </gazebo>
-        <gazebo reference="gnss_link">
+        <gazebo reference="gps_link">
             <material>Gazebo/Blue</material>
         </gazebo>

Commit message: Disabled IMU auto ned2enu transform

File: src/state_estimation/urdf/robot.xacro (robot description, xacro)
@@ -416,5 +416,5 @@
             <origin xyz="0 0 0.0275" rpy="0 0 0" />
             <parent link="sensors_base_link" />
-            <child link="gps_link"/>
+            <child link="gnss_link"/>
         </joint>
         <link name="radar_link">
@@ -456,5 +456,5 @@
             </collision>
         </link>
-        <link name="gps_link">
+        <link name="gnss_link">
             <inertial>
                 <mass value="0.1"/>
@@ -484,5 +484,5 @@
             <material>Gazebo/Red</material>
         </gazebo>
-        <gazebo reference="gps_link">
+        <gazebo reference="gnss_link">
             <material>Gazebo/Blue</material>
         </gazebo>
